Commit message: Add configuration files for Gazebo simulation and controllers
- Created gazebo_params.yaml for Gazebo parameters.
- Added my_controllers.yaml for controller configurations.
- Updated robot.urdf.xacro to conditionally include control files.
- Modified robot_core.xacro to replace cylinder with sphere for collision geometry.
- Introduced ros2_control.xacro for ROS 2 control integration.
- Enhanced launch files to support new parameters and spawner nodes.

File: description/robot.urdf.xacro (robot description, xacro)
@@ -1,6 +1,12 @@
 <?xml version="1.0"?>
 <robot xmlns:xacro="http://www.ros.org/wiki/xacro"  name="robot">
+    <xacro:arg name="use_ros2_control" default="true"/>
     <xacro:include filename="robot_core.xacro" />
-    <xacro:include filename="gazebo_control.xacro"/>
+    <xacro:if value="$(arg use_ros2_control)">
+        <xacro:include filename="ros2_control.xacro"/>
+    </xacro:if>
+    <xacro:unless value="$(arg use_ros2_control)">
+        <xacro:include filename="gazebo_control.xacro"/>
+    </xacro:unless>
     <xacro:include filename="lidar.xacro"/>
 </robot>

File: description/robot_core.xacro (robot description, xacro)
@@ -57,5 +57,5 @@
         <collision>
             <geometry>
-                <cylinder radius="0.078" length="0.035"/>
+                <sphere radius="0.078"/>
             </geometry>
         </collision>
@@ -83,5 +83,5 @@
         <collision>
             <geometry>
-                <cylinder radius="0.078" length="0.035"/>
+                <sphere radius="0.078"/>
             </geometry>
         </collision>
