Commit message: Gazebo-ROS2 linked, Lidar OK, impossible yo move the robot, looking for solutions but not found

File: description/gazebo_control.xacro (robot description, xacro)
@@ -2,20 +2,28 @@
 <robot xmlns:xacro="http://www.ros.org/wiki/xacro"  name="robot">
 <gazebo>
-    <plugin name="diff_drive" filename="libgazebo_ros_diffdrive.so">
+    <plugin name="gz::sim::systems::DiffDrive" filename="gz-sim-diff-drive-system">
         <!-- Wheel Information -->
         <left_joint>left_wheel_joint</left_joint>
         <right_joint>right_wheel_joint</right_joint>
-        <wheel_separation>0.35</wheel_separation>
-        <wheel_diameter>0.1</wheel_diameter>
+        <wheel_separation>0.535</wheel_separation>
+        <wheel_radius>0.078</wheel_radius>
         <!-- Limits -->
-        <max_wheel_torque>200</max_wheel_torque>
-        <max_wheel_acceleration>10.0</max_wheel_acceleration>
+         <!-- <max_wheel_torque>200</max_wheel_torque> -->
+        <max_linear_acceleration>0.33</max_linear_acceleration>
+        <!-- Input -->
+        <topic>cmd_vel</topic>
         <!-- Output -->
-        <odometry_frame>odom</odometry_frame>
-        <robot_base_frame>base_link</robot_base_frame>
-        <publish_odom>true</publish_odom>
-        <publish_odom_tf>true</publish_odom_tf>
-        <publish_wheel_tf>true</publish_wheel_tf>
+            <frame_id>odom</frame_id>
+            <child_frame_id>base_link</child_frame_id>
+            <odom_topic>odom</odom_topic>
+            <odom_publisher_frequency>30</odom_publisher_frequency>
+            <tf_topic>/tf</tf_topic>
     </plugin>
+        <plugin filename="gz-sim-joint-state-publisher-system"
+            name="gz::sim::systems::JointStatePublisher">
+            <topic>joint_states</topic>
+            <joint_name>left_wheel_joint</joint_name>
+            <joint_name>right_wheel_joint</joint_name>
+        </plugin>
 </gazebo>
 </robot>

File: description/lidar.xacro (robot description, xacro)
@@ -24,12 +24,12 @@
     <gazebo reference="laser_frame">
         <material>Gazebo/Red</material>
-        <sensor name="laser" type="ray">
+        <sensor name="laser" type="gpu_lidar">
             <pose> 0 0 0 0 0 0 </pose>
             <visualize>true</visualize>
             <update_rate>10</update_rate>
-            <ray>
+            <lidar>
                 <scan>
                     <horizontal>
-                        <samples>2250</samples>
+                        <samples>360</samples>
                         <min_angle>-2.356</min_angle>
                         <max_angle>2.356</max_angle>
@@ -40,12 +40,7 @@
                     <max>40</max>
                 </range>
-            </ray>
-            <plugin name="laser_controller" filename="libgazebo_ros_ray_sensor.so">
-                <ros>
-                    <argument>~/out:=scan</argument>
-                </ros>
-                <output_type>sensor_msgs/LaserScan</output_type>
-                <frame_name>laser_frame</frame_name>
-            </plugin>
+            </lidar>
+            <topic>scan</topic>
+             <gz_frame_id>laser_frame</gz_frame_id>
         </sensor>
     </gazebo>

File: description/robot.urdf.xacro (robot description, xacro)
@@ -2,4 +2,5 @@
 <robot xmlns:xacro="http://www.ros.org/wiki/xacro"  name="robot">
     <xacro:arg name="use_ros2_control" default="true"/>
+    <xacro:arg name="sim_mode" default="false"/>
     <xacro:include filename="robot_core.xacro" />
     <xacro:if value="$(arg use_ros2_control)">

File: description/robot_core.xacro (robot description, xacro)
@@ -57,5 +57,5 @@
         <collision>
             <geometry>
-                <sphere radius="0.078"/>
+                <cylinder radius="0.078" length="0.035"/>
             </geometry>
         </collision>
@@ -83,5 +83,5 @@
         <collision>
             <geometry>
-                <sphere radius="0.078"/>
+                <cylinder radius="0.078" length="0.035"/>
             </geometry>
         </collision>

File: description/ros2_control.xacro (robot description, xacro)
@@ -1,29 +1,32 @@
 <?xml version="1.0"?>
 <robot xmlns:xacro="http://www.ros.org/wiki/xacro"  name="robot">
-    <ros2_control name="GazeboSystem" type="system">
-        <hardware>
-            <plugin>gazebo_ros2_control/GazeboSystem</plugin>
-        </hardware>
-        <joint name="left_wheel_joint">
-            <command_interface name="velocity">
-                <param name="min">-10</param>
-                <param name="max">10</param>
-            </command_interface>
-            <state_interface name="velocity"/>
-            <state_interface name="position"/>
-        </joint>
-        <joint name="right_wheel_joint">
-            <command_interface name="velocity">
-                <param name="min">-10</param>
-                <param name="max">10</param>
-            </command_interface>
-            <state_interface name="velocity"/>
-            <state_interface name="position"/>
-        </joint>
-    </ros2_control>
+    <xacro:if value="$(arg sim_mode)">
+        <ros2_control name="GazeboSystem" type="system">
+            <hardware>
+                <plugin>gz_ros2_control/GazeboSimSystem</plugin>
+            </hardware>
+            <joint name="left_wheel_joint">
+                <command_interface name="velocity">
+                    <param name="min">-10</param>
+                    <param name="max">10</param>
+                </command_interface>
+                <state_interface name="velocity"/>
+                <state_interface name="position"/>
+            </joint>
+            <joint name="right_wheel_joint">
+                <command_interface name="velocity">
+                    <param name="min">-10</param>
+                    <param name="max">10</param>
+                </command_interface>
+                <state_interface name="velocity"/>
+                <state_interface name="position"/>
+            </joint>
+        </ros2_control>
+    </xacro:if>
     <gazebo>
-    <plugin name="diff_drive" filename="libgazebo_ros2_control.so">
+        <plugin name="gz_ros2_control::GazeboSimROS2ControlPlugin" filename="libgz_ros2_control-system.so">
             <parameters>$(find amr)/config/my_controllers.yaml</parameters>
-    </plugin>
-</gazebo>
+            <parameters>$(find amr)/config/gaz_ros2_ctl_use_sim.yaml</parameters>
+        </plugin>
+    </gazebo>
 </robot>
