Commit message: Moving, SLAM, NAV2

File: description/lidar.xacro (robot description, xacro)
@@ -37,5 +37,5 @@
                 </scan>
                 <range>
-                    <min>0.05</min>
+                    <min>0.5</min>
                     <max>40</max>
                 </range>

File: description/robot_core.xacro (robot description, xacro)
@@ -13,4 +13,12 @@
     <!-- BASE LINK -->
     <link name="base_link">
+    </link>
+    <!-- BASE_FOOTPRINT LINK-->
+    <joint name="base_footprint_joint" type="fixed">
+        <parent link="base_link"/>
+        <child link="base_footprint"/>
+        <origin xyz="0 0 0" rpy="0 0 0"/>
+    </joint>
+    <link name="base_footprint">
     </link>
     <!-- CHASSIS LINK -->
